Commit message: Turret (pan-tilt-camera) fully integrated and controllable

File: src/description/urdf/robot_base.xacro (robot description, xacro)
@@ -88,10 +88,91 @@
       <origin xyz="0.11 0 0.22"/>
     </joint>
-    <link name="camera_link"/>
-    <joint name="camera_joint" type="fixed">
-      <parent link="base_link"/>
-      <child link="camera_link"/>
-      <origin xyz="0.15 0 2" rpy="0 0.4 0"/>
-    </joint>
+    <!-- ================= PAN LINK ================= -->
+<link name="pan_link">
+  <visual>
+    <geometry>
+      <cylinder radius="0.05" length="0.02"/>
+    </geometry>
+    <material name="red">
+      <color rgba="1 0 0 1"/>
+    </material>
+  </visual>
+  <collision>
+    <geometry>
+      <cylinder radius="0.05" length="0.02"/>
+    </geometry>
+  </collision>
+  <inertial>
+    <mass value="0.5"/>
+    <origin xyz="0 0 0"/>
+    <inertia ixx="0.01" iyy="0.01" izz="0.01"
+             ixy="0" ixz="0" iyz="0"/>
+  </inertial>
+</link>
+<joint name="pan_joint" type="revolute">
+  <parent link="base_link"/>
+  <child link="pan_link"/>
+  <origin xyz="0.20 0 0.22"/>
+  <axis xyz="0 0 1"/>
+  <limit lower="-3.14" upper="3.14" effort="5" velocity="1"/>
+  <dynamics damping="0.1" friction="0.1"/>
+</joint>
+<!-- ================= TILT LINK ================= -->
+<link name="tilt_link">
+  <visual>
+    <geometry>
+      <box size="0.04 0.04 0.02"/>
+    </geometry>
+    <material name="black">
+      <color rgba="0.1 0.1 0.1 1"/>
+    </material>
+  </visual>
+  <collision>
+    <geometry>
+      <box size="0.04 0.04 0.02"/>
+    </geometry>
+  </collision>
+  <inertial>
+    <mass value="0.3"/>
+    <origin xyz="0 0 0"/>
+    <inertia ixx="0.005" iyy="0.005" izz="0.005"
+             ixy="0" ixz="0" iyz="0"/>
+  </inertial>
+</link>
+<joint name="tilt_base_joint" type="revolute">
+  <parent link="pan_link"/>
+  <child link="tilt_link"/>
+  <origin xyz="0 0 0.05"/>
+  <axis xyz="0 1 0"/>
+  <limit lower="-1.57" upper="1.57" effort="5" velocity="1"/>
+  <dynamics damping="0.1" friction="0.1"/>
+</joint>
+<!-- ================= CAMERA ================= -->
+<link name="camera_link">
+  <visual>
+    <geometry>
+      <box size="0.05 0.05 0.05"/>
+    </geometry>
+    <material name="red">
+      <color rgba="1 0 0 1"/>
+    </material>
+  </visual>
+  <collision>
+    <geometry>
+      <box size="0.05 0.05 0.05"/>
+    </geometry>
+  </collision>
+  <inertial>
+    <mass value="0.3"/>
+    <origin xyz="0 0 0"/>
+    <inertia ixx="0.005" iyy="0.005" izz="0.005"
+             ixy="0" ixz="0" iyz="0"/>
+  </inertial>
+</link>
+<joint name="camera_joint" type="fixed">
+  <parent link="tilt_link"/>
+  <child link="camera_link"/>
+  <origin xyz="0 0 0.03"/>
+</joint>
     <xacro:macro name="wheel" params="name x y">
       <link name="${name}_link">

Commit message: Added turret repositioning and side camera integration

File: src/description/urdf/robot_base.xacro (robot description, xacro)
@@ -86,5 +86,5 @@
       <parent link="base_link"/>
       <child link="lidar_link"/>
-      <origin xyz="0.11 0 0.22"/>
+      <origin xyz="0.22 0 0.22"/>
     </joint>
     <!-- ================= PAN LINK ================= -->
@@ -113,5 +113,5 @@
   <parent link="base_link"/>
   <child link="pan_link"/>
-  <origin xyz="0.20 0 0.22"/>
+  <origin xyz="0.12 0 0.21"/>
   <axis xyz="0 0 1"/>
   <limit lower="-3.14" upper="3.14" effort="5" velocity="1"/>
@@ -174,4 +174,31 @@
   <child link="camera_link"/>
   <origin xyz="0 0 0.03"/>
+</joint>
+<!-- ================= SIDE CAMERA ================= -->
+<link name="side_camera_link">
+  <visual>
+    <geometry>
+      <box size="0.05 0.05 0.05"/>
+    </geometry>
+    <material name="red">
+      <color rgba="1 0 0 1"/>
+    </material>
+  </visual>
+  <collision>
+    <geometry>
+      <box size="0.05 0.05 0.05"/>
+    </geometry>
+  </collision>
+  <inertial>
+    <mass value="0.3"/>
+    <origin xyz="0 0 0"/>
+    <inertia ixx="0.005" iyy="0.005" izz="0.005"
+             ixy="0" ixz="0" iyz="0"/>
+  </inertial>
+</link>
+<joint name="side_camera_joint" type="fixed">
+  <parent link="base_link"/>
+  <child link="side_camera_link"/>
+  <origin xyz="0.18 0.12 0.19"/>
 </joint>
     <xacro:macro name="wheel" params="name x y">

File: src/description/urdf/robot_sensors.xacro (robot description, xacro)
@@ -59,4 +59,23 @@
       </sensor>
     </gazebo>
+    <gazebo reference="side_camera_link">
+  <sensor name="side_camera_sensor" type="camera">
+    <always_on>true</always_on>
+    <update_rate>30</update_rate>
+    <topic>/side_camera/image_raw</topic>
+    <camera>
+      <horizontal_fov>1.047</horizontal_fov>
+      <image>
+        <width>640</width>
+        <height>480</height>
+        <format>R8G8B8</format>
+      </image>
+      <clip>
+        <near>0.1</near>
+        <far>100</far>
+      </clip>
+    </camera>
+  </sensor>
+</gazebo>
   </xacro:macro>
 </robot>

Commit message: Fixed side camera positioning and added proper bridge integration

File: src/description/urdf/robot_base.xacro (robot description, xacro)
@@ -200,5 +200,5 @@
   <parent link="base_link"/>
   <child link="side_camera_link"/>
-  <origin xyz="0.18 0.12 0.19"/>
+  <origin xyz="0.18 0.12 0.22"/>
 </joint>
     <xacro:macro name="wheel" params="name x y">
